File: _saved_mainboard.sch (KiCad schematic (older format))
At the start: 65 parts, among them J1 Screw_Terminal_1x02, J2 SERVO 5V, J3 Screw_Terminal_1x02, J4 Screw_Terminal_1x02, Q1 IRLR024NPBF, Q2 IRLR024NPBF, Q3 IRLR024NPBF, U1 AT90CAN128-16MU, U2 MCP2551-I/SN, Y1 Crystal

Commit message: Added mosfet and servo
Parts:
- gave numbers to parts that had none: 1
