File: mainboard.sch (KiCad schematic (older format))
At the start: 65 parts, among them J1 Screw_Terminal_1x02, J2 SERVO 5V, J3 Screw_Terminal_1x02, J4 Screw_Terminal_1x02, Q1 IRLR024NPBF, Q2 IRLR024NPBF, Q3 IRLR024NPBF, U1 AT90CAN128-16MU, U2 MCP2551-I/SN, Y1 Crystal

Commit message: Modified alot of stuff, added module and power for servo
Parts:
- removed C12: 100u, Capacitors_THT:CP_Radial_D7.5mm_P2.50mm, symbol CP1
- removed C13: 100u, Capacitors_SMD:CP_Elec_6.3x4.5, symbol CP1
- removed D3, D4: STTH2R06U, Diodes_SMD:D_SMA, symbol 1N4001
- removed J3, J4: Screw_Terminal_1x02, Connectors_Terminal_Blocks:TerminalBlock_Pheonix_MPT-2.54mm_2pol, symbol Screw_Terminal_1x02
- removed Q2, Q3: IRLR024NPBF, TO_SOT_Packages_SMD:TO-252-2, symbol IRLIZ44N
- removed R10: 10K, Resistors_SMD:R_1206, symbol R
- added D3: LED, LEDs:LED_1206, symbol LED
- added U3: EP_MODULE, EP_Module:EP_Module, symbol EP_MODULE
- R9: value 10K -> 1K
- gave numbers to parts that had none: 1
Connections:
- wire segments 292 -> 208
Other:
- note added: "Input servo 5V\n\n\n\n"
- note added: "Main Board - Electropioneer"
- note removed: "+"
- note removed: "-"
- note removed: "12V/5V"
- note removed: "PORTG pinouts\n\n"
- moved on the sheet: C11, C4, C5, C6, C7, C8, C9, D2, J2, PF1, PF_GND1, R6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

Commit message: Small modifs, but important
Connections:
- net GND: no longer D1.1 (K)
- net at R7.2: no longer D1.2 (A)
Changed lines of the file:
@@
 	2100 5300 2050 5300
 Wire Wire Line
-	2050 5200 2050 5300
-Wire Wire Line
-	1650 5200 2050 5200
+	2050 5300 2050 5200
+Wire Wire Line
+	2050 5200 1650 5200
 Wire Wire Line
 	1700 4950 1700 5550
@@
 Wire Wire Line
 	13400 900  13400 950
-Wire Wire Line
-	13400 1250 13400 1400
-Wire Wire Line
-	13400 1800 13400 1700
 Wire Wire Line
 	11400 850  11350 850
@@
 	11500 4150 11450 4150
 Wire Wire Line
-	11450 4400 11450 4150
-Wire Wire Line
-	10950 4400 11450 4400
+	11450 4150 11450 4400
+Wire Wire Line
+	11450 4400 10950 4400
 Wire Wire Line
 	11250 4400 11250 4450
@@
 Text Notes 11850 10150 0    118  ~ 0
 Main Board - Electropioneer
+Wire Wire Line
+	13400 1250 13400 1350
+Wire Wire Line
+	13400 1750 13400 1800
 $EndSCHEMATC

Commit message: Changed some footprints from 0603 t 0805
Parts:
- C1, C2, C6, C7, C8: footprint Capacitors_SMD:C_1206 -> Capacitors_SMD:C_0805
- D1, D2, D3: footprint LEDs:LED_1206 -> LEDs:LED_0805
- R1, R2, R3, R4, R5, R7, R8, R9: footprint Resistors_SMD:R_1206 -> Resistors_SMD:R_0805
Connections:
- net GND: now also D1.1 (K), D3.1 (K)
- net at R8.2: now also D2.2 (A)
- net at R7.2: now also D1.2 (A)
- net at R9.2: now also D3.2 (A)
Changed lines of the file:
@@
 LIBS:actel
 LIBS:analog_devices
+LIBS:bbd
+LIBS:bosch
 LIBS:brooktre
 LIBS:cmos_ieee
@@
 LIBS:microchip_pic18mcu
 LIBS:microchip_pic32mcu
+LIBS:modules
 LIBS:motor_drivers
 LIBS:msp430
 LIBS:nordicsemi
+LIBS:nxp
 LIBS:nxp_armmcu
 LIBS:onsemi
@@
 LIBS:switches
 LIBS:transf
+LIBS:triac_thyristor
 LIBS:ttl_ieee
 LIBS:video
+LIBS:wiznet
+LIBS:zetex
 LIBS:ep_module
 LIBS:mainboard-cache
@@
 F 0 "C2" H 1725 5800 50  0000 L CNN
 F 1 "33pF" H 1725 5600 50  0000 L CNN
-F 2 "Capacitors_SMD:C_1206" H 1738 5550 50  0001 C CNN
+F 2 "Capacitors_SMD:C_0805" H 1738 5550 50  0001 C CNN
 F 3 "" H 1700 5700 50  0001 C CNN
 	1    1700 5700
@@
 F 0 "C1" H 1325 5800 50  0000 L CNN
 F 1 "33pF" H 1325 5600 50  0000 L CNN
-F 2 "Capacitors_SMD:C_1206" H 1338 5550 50  0001 C CNN
+F 2 "Capacitors_SMD:C_0805" H 1338 5550 50  0001 C CNN
 F 3 "" H 1300 5700 50  0001 C CNN
 	1    1300 5700
@@
 F 0 "R5" V 12880 1100 50  0000 C CNN
 F 1 "10K" V 12800 1100 50  0000 C CNN
-F 2 "Resistors_SMD:R_1206" V 12730 1100 50  0001 C CNN
+F 2 "Resistors_SMD:R_0805" V 12730 1100 50  0001 C CNN
 F 3 "" H 12800 1100 50  0001 C CNN
 	1    12800 1100
@@
 F 0 "R7" V 13480 1100 50  0000 C CNN
 F 1 "1K" V 13400 1100 50  0000 C CNN
-F 2 "Resistors_SMD:R_1206" V 13330 1100 50  0001 C CNN
+F 2 "Resistors_SMD:R_0805" V 13330 1100 50  0001 C CNN
 F 3 "" H 13400 1100 50  0001 C CNN
 	1    13400 1100
@@
 F 0 "D1" H 13400 1650 50  0000 C CNN
 F 1 "LED" H 13400 1450 50  0000 C CNN
-F 2 "LEDs:LED_1206" H 13400 1550 50  0001 C CNN
+F 2 "LEDs:LED_0805" H 13400 1550 50  0001 C CNN
 F 3 "" H 13400 1550 50  0001 C CNN
 	1    13400 1550
@@
 F 0 "R4" V 2880 1900 50  0000 C CNN
 F 1 "120" V 2800 1900 50  0000 C CNN
-F 2 "Resistors_SMD:R_1206" V 2730 1900 50  0001 C CNN
+F 2 "Resistors_SMD:R_0805" V 2730 1900 50  0001 C CNN
 F 3 "" H 2800 1900 50  0001 C CNN
 	1    2800 1900
@@
 F 0 "R3" V 1480 2150 50  0000 C CNN
 F 1 "10K" V 1400 2150 50  0000 C CNN
-F 2 "Resistors_SMD:R_1206" V 1330 2150 50  0001 C CNN
+F 2 "Resistors_SMD:R_0805" V 1330 2150 50  0001 C CNN
 F 3 "" H 1400 2150 50  0001 C CNN
 	1    1400 2150
@@
 F 0 "R1" V 1180 1150 50  0000 C CNN
 F 1 "1K" V 1100 1150 50  0000 C CNN
-F 2 "Resistors_SMD:R_1206" V 1030 1150 50  0001 C CNN
+F 2 "Resistors_SMD:R_0805" V 1030 1150 50  0001 C CNN
 F 3 "" H 1100 1150 50  0001 C CNN
 	1    1100 1150
@@
 F 0 "R2" V 1280 1150 50  0000 C CNN
 F 1 "1K" V 1200 1150 50  0000 C CNN
-F 2 "Resistors_SMD:R_1206" V 1130 1150 50  0001 C CNN
+F 2 "Resistors_SMD:R_0805" V 1130 1150 50  0001 C CNN
 F 3 "" H 1200 1150 50  0001 C CNN
 	1    1200 1150
@@
 F 0 "C6" H 4475 1100 50  0000 L CNN
 F 1 "100n" H 4475 900 50  0000 L CNN
-F 2 "Capacitors_SMD:C_1206" H 4488 850 50  0001 C CNN
+F 2 "Capacitors_SMD:C_0805" H 4488 850 50  0001 C CNN
 F 3 "" H 4450 1000 50  0001 C CNN
 	1    4450 1000
@@
 F 0 "C7" H 4725 1100 50  0000 L CNN
 F 1 "100n" H 4725 900 50  0000 L CNN
-F 2 "Capacitors_SMD:C_1206" H 4738 850 50  0001 C CNN
+F 2 "Capacitors_SMD:C_0805" H 4738 850 50  0001 C CNN
 F 3 "" H 4700 1000 50  0001 C CNN
 	1    4700 1000
@@
 F 0 "C8" H 4975 1100 50  0000 L CNN
 F 1 "100n" H 4975 900 50  0000 L CNN
-F 2 "Capacitors_SMD:C_1206" H 4988 850 50  0001 C CNN
+F 2 "Capacitors_SMD:C_0805" H 4988 850 50  0001 C CNN
 F 3 "" H 4950 1000 50  0001 C CNN
 	1    4950 1000
@@
 F 0 "R8" V 15930 1100 50  0000 C CNN
 F 1 "1K" V 15850 1100 50  0000 C CNN
-F 2 "Resistors_SMD:R_1206" V 15780 1100 50  0001 C CNN
+F 2 "Resistors_SMD:R_0805" V 15780 1100 50  0001 C CNN
 F 3 "" H 15850 1100 50  0001 C CNN
 	1    15850 1100
@@
 F 0 "D2" H 15850 1600 50  0000 C CNN
 F 1 "LED" H 15850 1400 50  0000 C CNN
-F 2 "LEDs:LED_1206" H 15850 1500 50  0001 C CNN
+F 2 "LEDs:LED_0805" H 15850 1500 50  0001 C CNN
 F 3 "" H 15850 1500 50  0001 C CNN
 	1    15850 1500
@@
 F 0 "R9" V 11280 3900 50  0000 C CNN
 F 1 "1K" V 11200 3900 50  0000 C CNN
-F 2 "Resistors_SMD:R_1206" V 11130 3900 50  0001 C CNN
+F 2 "Resistors_SMD:R_0805" V 11130 3900 50  0001 C CNN
 F 3 "" H 11200 3900 50  0001 C CNN
 	1    11200 3900
@@
 F 0 "D3" H 10950 4250 50  0000 C CNN
 F 1 "LED" H 10950 4050 50  0000 C CNN
-F 2 "LEDs:LED_1206" H 10950 4150 50  0001 C CNN
+F 2 "LEDs:LED_0805" H 10950 4150 50  0001 C CNN
 F 3 "" H 10950 4150 50  0001 C CNN
 	1    10950 4150
@@
 	11050 3900 10950 3900
 Wire Wire Line
-	10950 3900 10950 3950
+	10950 3900 10950 4000
 Wire Wire Line
 	11500 4150 11450 4150
@@
 	11250 4400 11250 4450
 Wire Wire Line
-	10950 4400 10950 4350
+	10950 4400 10950 4300
 Connection ~ 11250 4400
 Wire Wire Line
-	15850 1250 15850 1300
+	15850 1250 15850 1350
 Wire Wire Line
 	3850 2100 3900 2100
@@
 Main Board - Electropioneer
 Wire Wire Line
-	13400 1250 13400 1350
-Wire Wire Line
-	13400 1750 13400 1800
+	13400 1250 13400 1400
+Wire Wire Line
+	13400 1700 13400 1800
 $EndSCHEMATC

Commit message: Added EP_Module to glavna
Parts:
- U2: symbol MCP2551-I/SN -> MCP2551-I/SN-RESCUE-mainboard
Changed lines of the file:
@@
 LIBS:ac-dc
 LIBS:actel
+LIBS:allegro
 LIBS:analog_devices
+LIBS:battery_management
 LIBS:bbd
 LIBS:bosch
@@
 LIBS:hc11
 LIBS:ir
+LIBS:leds
 LIBS:logo
 LIBS:maxim
+LIBS:mechanical
 LIBS:microchip_dspic33dsc
 LIBS:microchip_pic10mcu
@@
 LIBS:microchip_pic16mcu
 LIBS:microchip_pic18mcu
+LIBS:microchip_pic24mcu
 LIBS:microchip_pic32mcu
 LIBS:modules
 LIBS:motor_drivers
+LIBS:motors
 LIBS:msp430
 LIBS:nordicsemi
@@
 LIBS:wiznet
 LIBS:zetex
-LIBS:ep_module
 LIBS:mainboard-cache
 EELAYER 25 0
@@
 $EndComp
 $Comp
-L MCP2551-I/SN U2
+L MCP2551-I/SN-RESCUE-mainboard U2
 U 1 1 59594AC0
 P 1950 1600
